File: kicad/lownoise-pwr.sch (KiCad schematic (older format))
At the start: 25 parts, among them J1 Conn_01x02_Female, J2 Conn_01x02_Female, J3 Conn_01x02_Female, Q1 BD244C, U1 LM723_DIP14, U2 LM4040DBZ-4.1

Commit message: Starts long way to screw-plugs
Parts:
- removed J2: Conn_01x02_Female, Connector_PinHeader_2.54mm:PinHeader_1x02_P2.54mm_Vertical, symbol Connector:Conn_01x02_Female
- added J2: Conn_01x02_Female, TerminalBlock_Phoenix:TerminalBlock_Phoenix_MKDS-3-2-5.08_1x02_P5.08mm_Horizontal, symbol Connector:Screw_Terminal_01x02
- F1: footprint Fuse:Fuseholder_Cylinder-5x20mm_Schurter_0031_8201_Horizontal_Open -> Fuse:Fuse_Bourns_MF-RHT1000
- J1: footprint Connector_PinHeader_2.54mm:PinHeader_1x02_P2.54mm_Vertical -> TerminalBlock_Phoenix:TerminalBlock_Phoenix_MKDS-3-2-5.08_1x02_P5.08mm_Horizontal; symbol Connector:Conn_01x02_Female -> Connector:Screw_Terminal_01x02
Connections:
- net GND: now also J2.1 (Pin_1)
- net at C6.1, C8.1, R4.1: now also J2.2 (Pin_2)
Changed lines of the file:
@@
-$EndComp
-$Comp
-L Connector:Conn_01x02_Female J2
-U 1 1 5E2092FB
-P 8250 2050
-F 0 "J2" H 8278 2026 50  0000 L CNN
-F 1 "Conn_01x02_Female" H 8278 1935 50  0000 L CNN
-F 2 "Connector_PinHeader_2.54mm:PinHeader_1x02_P2.54mm_Vertical" H 8250 2050 50  0001 C CNN
-F 3 "~" H 8250 2050 50  0001 C CNN
-	1    8250 2050
-	1    0    0    -1
 $EndComp
 $Comp
@@
 F 0 "F1" H 3210 2546 50  0000 L CNN
 F 1 "Fuse" H 3210 2455 50  0000 L CNN
-F 2 "Fuse:Fuseholder_Cylinder-5x20mm_Schurter_0031_8201_Horizontal_Open" V 3080 2500 50  0001 C CNN
+F 2 "Fuse:Fuse_Bourns_MF-RHT1000" V 3080 2500 50  0001 C CNN
 F 3 "~" H 3150 2500 50  0001 C CNN
 	1    3150 2500
@@
 $EndComp
 $Comp
-L Connector:Conn_01x02_Female J1
+L Connector:Screw_Terminal_01x02 J1
 U 1 1 5E20A2EE
 P 2800 2500
 F 0 "J1" H 2750 2600 50  0000 C CNN
 F 1 "Conn_01x02_Female" H 2650 2300 50  0000 C CNN
-F 2 "Connector_PinHeader_2.54mm:PinHeader_1x02_P2.54mm_Vertical" H 2800 2500 50  0001 C CNN
+F 2 "TerminalBlock_Phoenix:TerminalBlock_Phoenix_MKDS-3-2-5.08_1x02_P5.08mm_Horizontal" V 3250 2500 50  0000 C CNN
 F 3 "~" H 2800 2500 50  0001 C CNN
 	1    2800 2500
@@
 Wire Wire Line
 	4100 3600 4100 4000
+$Comp
+L Connector:Screw_Terminal_01x02 J2
+U 1 1 5F16A6BD
+P 8250 2150
+F 0 "J2" H 8200 2250 50  0000 C CNN
+F 1 "Conn_01x02_Female" H 8100 1950 50  0000 C CNN
+F 2 "TerminalBlock_Phoenix:TerminalBlock_Phoenix_MKDS-3-2-5.08_1x02_P5.08mm_Horizontal" V 8700 2150 50  0001 C CNN
+F 3 "~" H 8250 2150 50  0001 C CNN
+	1    8250 2150
+	1    0    0    1
+$EndComp
 $EndSCHEMATC

Commit message: Adds output screw-plugs, big transistor
R4 now vertical to gain space for screw-plugs
Input srew-plug not completely on PCB, soldered wires preferred
Adds 2nd via to solder polymer-fuse instead of glas fuseholder
Parts:
- F1: footprint Fuse:Fuse_Bourns_MF-RHT1000 -> Fuse:Fuseholder_Cylinder-5x20mm_Schurter_0031_8201_Horizontal_Open
- Q1: value BD244C -> BD244C / MJD6284; footprint Package_TO_SOT_THT:TO-220-3_Vertical -> Package_TO_SOT_THT:TO-247-3_Vertical
- R4: footprint Resistor_THT:R_Axial_DIN0516_L15.5mm_D5.0mm_P20.32mm_Horizontal -> Resistor_THT:R_Axial_DIN0516_L15.5mm_D5.0mm_P5.08mm_Vertical
Changed lines of the file:
@@
 P 5450 2150
 F 0 "Q1" V 5779 2150 50  0000 C CNN
-F 1 "BD244C" V 5688 2150 50  0000 C CNN
-F 2 "Package_TO_SOT_THT:TO-220-3_Vertical" H 5655 2070 50  0001 L CIN
+F 1 "BD244C / MJD6284" V 5688 2150 50  0000 C CNN
+F 2 "Package_TO_SOT_THT:TO-247-3_Vertical" H 5655 2070 50  0001 L CIN
 F 3 "http://www.mospec.com.tw/pdf/power/BD249.pdf" H 5450 2150 50  0001 L CNN
 	1    5450 2150
@@
 F 0 "R4" V 6250 2050 50  0000 C CNN
 F 1 "2R7" V 6034 2050 50  0000 C CNN
-F 2 "Resistor_THT:R_Axial_DIN0516_L15.5mm_D5.0mm_P20.32mm_Horizontal" V 6080 2050 50  0001 C CNN
+F 2 "Resistor_THT:R_Axial_DIN0516_L15.5mm_D5.0mm_P5.08mm_Vertical" V 6080 2050 50  0001 C CNN
 F 3 "~" H 6150 2050 50  0001 C CNN
 	1    6150 2050
@@
 F 0 "F1" H 3210 2546 50  0000 L CNN
 F 1 "Fuse" H 3210 2455 50  0000 L CNN
-F 2 "Fuse:Fuse_Bourns_MF-RHT1000" V 3080 2500 50  0001 C CNN
+F 2 "Fuse:Fuseholder_Cylinder-5x20mm_Schurter_0031_8201_Horizontal_Open" V 3080 2500 50  0001 C CNN
 F 3 "~" H 3150 2500 50  0001 C CNN
 	1    3150 2500
@@
 F 0 "J1" H 2750 2600 50  0000 C CNN
 F 1 "Conn_01x02_Female" H 2650 2300 50  0000 C CNN
-F 2 "TerminalBlock_Phoenix:TerminalBlock_Phoenix_MKDS-3-2-5.08_1x02_P5.08mm_Horizontal" V 3250 2500 50  0000 C CNN
+F 2 "TerminalBlock_Phoenix:TerminalBlock_Phoenix_MKDS-3-2-5.08_1x02_P5.08mm_Horizontal" V 3250 2500 50  0001 C CNN
 F 3 "~" H 2800 2500 50  0001 C CNN
 	1    2800 2500

Commit message: Adds another C to ensure bigger capacity is possible
Reason: components local availability
Parts:
- added C9: 500n, Capacitor_THT:C_Disc_D5.0mm_W2.5mm_P2.50mm, symbol Device:C
- C4: value 1000n -> 500n
Connections:
- net GND: now also C9.2
- net at C2.1, C4.1, R1.1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: now also C9.1
Other:
- moved on the sheet: C2, R1, R2
Changed lines of the file:
@@
 L Device:R R2
 U 1 1 5E2166FF
-P 4450 3000
-F 0 "R2" H 4520 3046 50  0000 L CNN
-F 1 "1k" H 4520 2955 50  0000 L CNN
-F 2 "Resistor_THT:R_Axial_DIN0207_L6.3mm_D2.5mm_P7.62mm_Horizontal" V 4380 3000 50  0001 C CNN
-F 3 "~" H 4450 3000 50  0001 C CNN
-	1    4450 3000
-	1    0    0    -1
-$EndComp
-Wire Wire Line
-	4950 2850 4450 2850
+P 4500 3000
+F 0 "R2" H 4570 3046 50  0000 L CNN
+F 1 "1k" H 4570 2955 50  0000 L CNN
+F 2 "Resistor_THT:R_Axial_DIN0207_L6.3mm_D2.5mm_P7.62mm_Horizontal" V 4430 3000 50  0001 C CNN
+F 3 "~" H 4500 3000 50  0001 C CNN
+	1    4500 3000
+	1    0    0    -1
+$EndComp
+Wire Wire Line
+	4950 2850 4500 2850
 $Comp
 L Device:C C4
 U 1 1 5E218AAD
 P 4750 3650
-F 0 "C4" H 4865 3696 50  0000 L CNN
-F 1 "1000n" H 4865 3605 50  0000 L CNN
+F 0 "C4" H 4750 3750 50  0000 L CNN
+F 1 "500n" V 4800 3400 50  0000 L CNN
 F 2 "Capacitor_THT:C_Disc_D5.0mm_W2.5mm_P2.50mm" H 4788 3500 50  0001 C CNN
 F 3 "~" H 4750 3650 50  0001 C CNN
@@
 L Device:CP C2
 U 1 1 5E21BA6D
-P 4450 3650
-F 0 "C2" H 4200 3700 50  0000 L CNN
-F 1 "100u" H 4150 3600 50  0000 L CNN
-F 2 "Capacitor_THT:C_Radial_D8.0mm_H7.0mm_P3.50mm" H 4488 3500 50  0001 C CNN
-F 3 "~" H 4450 3650 50  0001 C CNN
-	1    4450 3650
+P 4250 3650
+F 0 "C2" H 4250 3750 50  0000 L CNN
+F 1 "100u" V 4300 3400 50  0000 L CNN
+F 2 "Capacitor_THT:C_Radial_D8.0mm_H7.0mm_P3.50mm" H 4288 3500 50  0001 C CNN
+F 3 "~" H 4250 3650 50  0001 C CNN
+	1    4250 3650
 	1    0    0    -1
 $EndComp
@@
 L power:GND #PWR04
 U 1 1 5E21C3CE
-P 4450 4000
-F 0 "#PWR04" H 4450 3750 50  0001 C CNN
-F 1 "GND" H 4455 3827 50  0000 C CNN
-F 2 "" H 4450 4000 50  0001 C CNN
-F 3 "" H 4450 4000 50  0001 C CNN
-	1    4450 4000
+P 4250 4000
+F 0 "#PWR04" H 4250 3750 50  0001 C CNN
+F 1 "GND" H 4255 3827 50  0000 C CNN
+F 2 "" H 4250 4000 50  0001 C CNN
+F 3 "" H 4250 4000 50  0001 C CNN
+	1    4250 4000
 	1    0    0    -1
 $EndComp
@@
 $EndComp
 Wire Wire Line
-	4450 3150 4450 3500
-Connection ~ 4450 3150
-Wire Wire Line
-	4450 3150 4750 3150
+	4250 3150 4250 3500
 Wire Wire Line
 	4750 3150 4750 3500
@@
 L Device:R_POT_Small R1
 U 1 1 5E657629
-P 4100 3400
-F 0 "R1" H 4040 3446 50  0000 R CNN
-F 1 "4k7" H 4040 3355 50  0000 R CNN
-F 2 "Potentiometer_THT:Potentiometer_Bourns_3296W_Vertical" V 4030 3400 50  0001 C CNN
-F 3 "~" H 4100 3400 50  0001 C CNN
-	1    4100 3400
+P 3900 3400
+F 0 "R1" H 3840 3446 50  0000 R CNN
+F 1 "4k7" H 3840 3355 50  0000 R CNN
+F 2 "Potentiometer_THT:Potentiometer_Bourns_3296W_Vertical" V 3830 3400 50  0001 C CNN
+F 3 "~" H 3900 3400 50  0001 C CNN
+	1    3900 3400
 	1    0    0    -1
 $EndComp
@@
 L power:GND #PWR02
 U 1 1 5E657FEF
-P 4100 4000
-F 0 "#PWR02" H 4100 3750 50  0001 C CNN
-F 1 "GND" H 4105 3827 50  0000 C CNN
-F 2 "" H 4100 4000 50  0001 C CNN
-F 3 "" H 4100 4000 50  0001 C CNN
-	1    4100 4000
-	1    0    0    -1
-$EndComp
-Wire Wire Line
-	4100 3150 4450 3150
+P 3900 4000
+F 0 "#PWR02" H 3900 3750 50  0001 C CNN
+F 1 "GND" H 3905 3827 50  0000 C CNN
+F 2 "" H 3900 4000 50  0001 C CNN
+F 3 "" H 3900 4000 50  0001 C CNN
+	1    3900 4000
+	1    0    0    -1
+$EndComp
+Wire Wire Line
+	3900 3150 4250 3150
 Connection ~ 7050 2050
 Wire Wire Line
@@
 	4750 4000 4750 3800
 Wire Wire Line
-	4450 3800 4450 4000
+	4250 3800 4250 4000
 Wire Wire Line
 	3600 3100 3600 4000
@@
 	6150 3500 6600 3500
 Wire Wire Line
-	4100 3500 4100 3600
-Wire Wire Line
-	4100 3150 4100 3300
-Wire Wire Line
-	4200 3400 4200 3600
-Wire Wire Line
-	4200 3600 4100 3600
-Connection ~ 4100 3600
-Wire Wire Line
-	4100 3600 4100 4000
+	3900 3500 3900 3600
+Wire Wire Line
+	3900 3150 3900 3300
+Wire Wire Line
+	4000 3400 4000 3600
+Wire Wire Line
+	4000 3600 3900 3600
+Connection ~ 3900 3600
+Wire Wire Line
+	3900 3600 3900 4000
 $Comp
 L Connector:Screw_Terminal_01x02 J2
@@
 	1    0    0    1
 $EndComp
+$Comp
+L Device:C C9
+U 1 1 5F7AA236
+P 4500 3650
+F 0 "C9" H 4500 3750 50  0000 L CNN
+F 1 "500n" V 4550 3400 50  0000 L CNN
+F 2 "Capacitor_THT:C_Disc_D5.0mm_W2.5mm_P2.50mm" H 4538 3500 50  0001 C CNN
+F 3 "~" H 4500 3650 50  0001 C CNN
+	1    4500 3650
+	1    0    0    -1
+$EndComp
+Wire Wire Line
+	4500 3500 4500 3150
+Connection ~ 4500 3150
+Wire Wire Line
+	4500 3150 4750 3150
+Connection ~ 4250 3150
+Wire Wire Line
+	4250 3150 4500 3150
+$Comp
+L power:GND #PWR014
+U 1 1 5F7C1931
+P 4500 4000
+F 0 "#PWR014" H 4500 3750 50  0001 C CNN
+F 1 "GND" H 4505 3827 50  0000 C CNN
+F 2 "" H 4500 4000 50  0001 C CNN
+F 3 "" H 4500 4000 50  0001 C CNN
+	1    4500 4000
+	1    0    0    -1
+$EndComp
+Wire Wire Line
+	4500 4000 4500 3800
 $EndSCHEMATC
